Commit message: Added Simplified Collision Meshes For Arm URDF to speed up simulation

File: rover/simulation/urdfs/2022_Arm_URDF.urdf (robot description, URDF)
Before this commit: robot 2022_Arm_URDF, 7 links, 6 joints
Links:
- link Link_1: geometry collision mesh filename=package://rover/rover/simulation/meshes/Arm_2022/Collision_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; visual mesh filename=package://rover/rover/simulation/meshes/Arm_2022/Link_1.STL
- link Link_2: geometry collision mesh filename=package://rover/rover/simulation/meshes/Arm_2022/Collision_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; visual mesh filename=package://rover/rover/simulation/meshes/Arm_2022/Link_2.STL
- link Link_3: geometry collision mesh filename=package://rover/rover/simulation/meshes/Arm_2022/Collision_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; visual mesh filename=package://rover/rover/simulation/meshes/Arm_2022/Link_3.STL
- link Link_4: geometry collision mesh filename=package://rover/rover/simulation/meshes/Arm_2022/Collision_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; visual mesh filename=package://rover/rover/simulation/meshes/Arm_2022/Link_4.STL
- link Link_5: geometry collision mesh filename=package://rover/rover/simulation/meshes/Arm_2022/Collision_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; visual mesh filename=package://rover/rover/simulation/meshes/Arm_2022/Link_5.STL
- link Link_6: geometry collision mesh filename=package://rover/rover/simulation/meshes/Arm_2022/Collision_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; visual mesh filename=package://rover/rover/simulation/meshes/Arm_2022/Link_6.STL
- link base_link: geometry collision mesh filename=package://rover/rover/simulation/meshes/Arm_2022/Collision_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; visual mesh filename=package://rover/rover/simulation/meshes/Arm_2022/base_link.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
