Commit message: arm_simulation.py can publish to /joint_states and move arm in rivz
- tested with old, hence modification to launch file
- renamed a joint in old arm urdf

File: rover/simulation/urdfs/Arm_2022_URDF.urdf (robot description, URDF)
Before this commit: robot Arm_2022_URDF, 7 links, 6 joints
Joints:
- removed joint Jont_1
- added joint Joint_1: type continuous, parent base_link, child Link_1, origin xyz=0.0634999999999999 0.0634999999999998 0.073885628993429 rpy=0 0 0, axis 0 0 1
