Commit message: This is the updated urdf file for robot base which has hector imu plugin and its orientation has been changed by 90 degrees to prevent error in z values of acceleration.

File: rover/simulation/urdfs/robot_base.urdf (robot description, URDF)
Before this commit: robot robot_base, 6 links, 5 joints
Joints:
- joint imu_joint: origin xyz=0.0 0 0.278189004081027 rpy=0 0 0 -> xyz=0.0 0 0.0 rpy=1.5707963267949 0 0

Commit message: This file has IMU, GPS and LIDAR integrated with odometry of IMU and GPS

File: rover/simulation/urdfs/robot_base.urdf (robot description, URDF)
Before this commit: robot robot_base, 7 links, 6 joints
Links:
- added link lidar_link, mass 0.425; collision mesh filename=package://mobile_manipulator_body/meshes/os1_64.stl; visual mesh filename=package://mobile_manipulator_body/meshes/os1_64.stl
Joints:
- added joint lidar_joint: type fixed, parent base_link, child lidar_link, origin xyz=0.0 0 0.278189004081027 rpy=0 0 0, axis 0 0 0

Commit message: adding updates to simulation with dummy robot base

File: rover/simulation/urdfs/robot_base.urdf (robot description, URDF)
Before this commit: robot robot_base, 8 links, 7 joints
Links:
- link base_link: geometry collision mesh filename=package://rover/rover/simulation/meshes/robot_base.stl; visual mesh filename=package://rover/rover/simulation/meshes/robot_base.stl
- link front_left_wheel: geometry collision mesh filename=package://rover/rover/simulation/meshes/wheel.stl; visual mesh filename=package://rover/rover/simulation/meshes/wheel.stl
- link front_right_wheel: geometry collision mesh filename=package://rover/rover/simulation/meshes/wheel.stl; visual mesh filename=package://rover/rover/simulation/meshes/wheel.stl
- link lidar_link: geometry collision mesh filename=package://rover/rover/simulation/meshes/os1_64.stl; visual mesh filename=package://rover/rover/simulation/meshes/os1_64.stl
- link rear_left_wheel: geometry collision mesh filename=package://rover/rover/simulation/meshes/wheel.stl; visual mesh filename=package://rover/rover/simulation/meshes/wheel.stl
- link rear_right_wheel: geometry collision mesh filename=package://rover/rover/simulation/meshes/wheel.stl; visual mesh filename=package://rover/rover/simulation/meshes/wheel.stl
