Commit message: Testing branch for local_planner

File: rover/simulation/urdfs/Rover.urdf (robot description, URDF)
Before this commit: robot rover, 12 links, 11 joints
Joints:
- joint gps_joint: origin xyz=0.0 0 0.278189004081027 rpy=0 0 0 -> xyz=0.280596630449412 0.391929398096866 0.278189004081027 rpy=0 0 0
- joint imu_joint: origin xyz=0.0 0 0.0 rpy=1.5707963267949 0 0 -> xyz=0.280596630449412 0.391929398096866 0.497299040946044 rpy=1.5707963267949 0 0
- joint lidar_joint: origin xyz=0.0 0 0.278189004081027 rpy=0 0 0 -> xyz=0.280596630449412 0.391929398096866 0.278189004081027 rpy=0 0 0
