Commit message: Got camera working on rviz and gazebo, point cloud data is funky

File: rover/simulation/urdfs/bruh_with_EE.xacro (robot description, xacro)
@@ -234,3 +234,21 @@
   <limit upper="0.0" lower="-0.04" effort="100" velocity="100"/>
 </joint>
+<link name="camera_link">
+  <visual>
+    <geometry>
+      <box size="0.01 0.01 0.05"/>
+    </geometry>
+    <material name="silver"/>
+  </visual>
+  <!-- <collision>
+    <geometry>
+      <box size="0.01 0.01 0.01"/>
+    </geometry>
+  </collision> -->
+</link>
+<joint name="camera_joint" type="fixed">
+  <parent link="Link_4"/>
+  <child link="camera_link"/>
+  <origin xyz="0 0.06 0.4" rpy="0 0 0"/> <!--red green blue-->
+</joint>
 </robot>

File: rover/simulation/urdfs/bruh_with_EE_gazebo.xacro (robot description, xacro)
@@ -321,5 +321,5 @@
   <child link="base_link"/>
 </joint>
-<!-- Gazebo Plugin -->
+<!-- Gazebo Plugins-->
 <gazebo>
   <plugin name ="gazebo_ros_control" filename="libgazebo_ros_control.so">
@@ -342,3 +342,70 @@
     </plugin>
 </gazebo>
+<!-- Gazebo Depth Camera -->
+<link name="camera_link">
+  <visual>
+    <origin xyz="0 0 0" rpy="0 0 0"/>
+    <geometry>
+      <box size="0.01 0.01 0.05"/>
+    </geometry>
+    <material name="red"/>
+  </visual>
+  <!-- <collision>
+    <geometry>
+      <box size="0.01 0.01 0.01"/>
+    </geometry>
+  </collision> -->
+</link>
+<link name="camera_optical"/>
+<joint name="camera_joint" type="fixed">
+  <parent link="Link_4"/>
+  <child link="camera_link"/>
+  <origin xyz="0 0.1 0.4" rpy="0 1.57 0"/> <!--red green blue-->
+</joint>
+<joint name="optical_joint" type="fixed">
+  <parent link="camera_link"/>
+  <child link="camera_optical"/>
+  <origin xyz="0 0 0" rpy="3.1415 0 0"/>
+</joint>
+<gazebo reference="camera_link">
+  <sensor name="camera" type="depth">
+    <update_rate>20</update_rate>
+    <camera>
+      <horizontal_fov>1.5</horizontal_fov>
+      <image>
+        <width>640</width>
+        <height>480</height>
+        <format>R8G8B8</format>
+      </image>
+      <clip>
+        <near>0.05</near>
+        <far>3</far>
+      </clip>
+    </camera>
+    <plugin name="camera_plugin" filename="libgazebo_ros_openni_kinect.so">
+      <baseline>0.2</baseline>
+      <alwaysOn>true</alwaysOn>
+      <updateRate>1.0</updateRate>
+      <cameraName>camera_ir</cameraName>
+      <imageTopicName>/camera/color/image_raw</imageTopicName>
+      <cameraInfoTopicName>/camera/color/camera_info</cameraInfoTopicName>
+      <depthImageTopicName>/camera/depth/image_raw</depthImageTopicName>
+      <depthImageInfoTopicName>/camera/depth/camera_info</depthImageInfoTopicName>
+      <pointCloudTopicName>/camera/depth/points</pointCloudTopicName>
+      <frameName>camera_optical</frameName> <!-- name of link -->
+      <pointCloudCutoff>0</pointCloudCutoff>
+      <pointCloudCutoffMax>3.5</pointCloudCutoffMax>
+      <distortionK1>0</distortionK1>
+      <distortionK2>0</distortionK2>
+      <distortionK3>0</distortionK3>
+      <distortionT1>0</distortionT1>
+      <distortionT2>0</distortionT2>
+      <CxPrime>0</CxPrime>
+      <Cx>0</Cx>
+      <Cy>0</Cy>
+      <focalLength>0</focalLength>
+      <hackBaseline>0</hackBaseline>
+    </plugin>
+  </sensor>
+</gazebo>
 </robot>
