Commit message: working end effector in gazebo, tho it doesn't grip, only launch

File: rover/simulation/urdfs/bruh_with_EE_gazebo.xacro (robot description, xacro)
@@ -104,5 +104,5 @@
   </collision>
 </link>
-<link name="Link_1"> <!-- turntable -->
+<link name="Link_1">
   <inertial>
     <origin xyz="-8.21703816100694e-14 -0.00019647994583754658 0.036488404975619185" rpy="0 0 0"/>
@@ -197,5 +197,5 @@
 </joint>
 <joint name="Joint_3" type="continuous">
-  <origin xyz="0.0 0.0 0.375" rpy="-1.57 0 0"/>
+  <origin xyz="0.0 0.0 0.375" rpy="0 0 0"/>
   <parent link="Link_2"/>
   <child link="Link_3"/>
@@ -234,3 +234,96 @@
   <limit upper="0.0" lower="-0.04" effort="100" velocity="100"/>
 </joint>
+<!-- URDF Transmissions-->
+<transmission name="tran1">
+  <type>transmission_interface/SimpleTransmission</type>
+  <joint name="Joint_1">
+      <hardwareInterface>PositionJointInterface</hardwareInterface>
+  </joint>
+  <actuator name="motor1">
+      <hardwareInterface>PositionJointInterface</hardwareInterface>
+      <mechanicalReduction>1</mechanicalReduction>
+  </actuator>
+</transmission>
+<transmission name="tran2">
+  <type>transmission_interface/SimpleTransmission</type>
+  <joint name="Joint_2">
+      <hardwareInterface>PositionJointInterface</hardwareInterface>
+  </joint>
+  <actuator name="motor2">
+      <hardwareInterface>PositionJointInterface</hardwareInterface>
+      <mechanicalReduction>1</mechanicalReduction>
+  </actuator>
+</transmission>
+<transmission name="tran3">
+  <type>transmission_interface/SimpleTransmission</type>
+  <joint name="Joint_3">
+      <hardwareInterface>PositionJointInterface</hardwareInterface>
+  </joint>
+  <actuator name="motor3">
+      <hardwareInterface>PositionJointInterface</hardwareInterface>
+      <mechanicalReduction>1</mechanicalReduction>
+  </actuator>
+</transmission>
+<transmission name="tran4">
+  <type>transmission_interface/SimpleTransmission</type>
+  <joint name="Joint_4">
+      <hardwareInterface>PositionJointInterface</hardwareInterface>
+  </joint>
+  <actuator name="motor4">
+      <hardwareInterface>PositionJointInterface</hardwareInterface>
+      <mechanicalReduction>1</mechanicalReduction>
+  </actuator>
+</transmission>
+<transmission name="tran5">
+  <type>transmission_interface/SimpleTransmission</type>
+  <joint name="Joint_5">
+      <hardwareInterface>PositionJointInterface</hardwareInterface>
+  </joint>
+  <actuator name="motor5">
+      <hardwareInterface>PositionJointInterface</hardwareInterface>
+      <mechanicalReduction>1</mechanicalReduction>
+  </actuator>
+</transmission>
+<transmission name="tran6">
+  <type>transmission_interface/SimpleTransmission</type>
+  <joint name="Joint_6">
+      <hardwareInterface>PositionJointInterface</hardwareInterface>
+  </joint>
+  <actuator name="motor6">
+      <hardwareInterface>PositionJointInterface</hardwareInterface>
+      <mechanicalReduction>1</mechanicalReduction>
+  </actuator>
+</transmission>
+<transmission name="tran7">
+  <type>transmission_interface/SimpleTransmission</type>
+  <joint name="Joint_7">
+      <hardwareInterface>PositionJointInterface</hardwareInterface>
+  </joint>
+  <actuator name="motor7">
+      <hardwareInterface>EffortJointInterface</hardwareInterface>
+      <mechanicalReduction>1</mechanicalReduction>
+  </actuator>
+</transmission>
+<transmission name="tran8">
+  <type>transmission_interface/SimpleTransmission</type>
+  <joint name="Joint_8">
+      <hardwareInterface>PositionJointInterface</hardwareInterface>
+  </joint>
+  <actuator name="motor8">
+      <hardwareInterface>EffortJointInterface</hardwareInterface>
+      <mechanicalReduction>1</mechanicalReduction>
+  </actuator>
+</transmission>
+<!-- Fix arm in place -->
+<link name="world"/>
+<joint name="fixed" type="fixed">
+  <parent link="world"/>
+  <child link="base_link"/>
+</joint>
+<!-- Gazebo Plugin -->
+<gazebo>
+  <plugin name ="gazebo_ros_control" filename="libgazebo_ros_control.so">
+    <robotNamespace>/arm</robotNamespace>
+  </plugin>
+</gazebo>
 </robot>

Commit message: synced gazebo depth camera with rviz

File: rover/simulation/urdfs/bruh_with_EE_gazebo.xacro (robot description, xacro)
@@ -359,12 +359,12 @@
 <link name="camera_optical"/>
 <joint name="camera_joint" type="fixed">
-  <parent link="Link_4"/>
+  <parent link="Link_6"/>
   <child link="camera_link"/>
-  <origin xyz="0 0.1 0.4" rpy="0 1.57 0"/> <!--red green blue-->
+  <origin xyz="0 0.1 0" rpy="1.571 -1.571 1.571"/> <!--red green blue-->
 </joint>
 <joint name="optical_joint" type="fixed">
   <parent link="camera_link"/>
   <child link="camera_optical"/>
-  <origin xyz="0 0 0" rpy="3.1415 0 0"/>
+  <origin xyz="0 0 0" rpy="-1.571 0 -1.571"/>
 </joint>
 <gazebo reference="camera_link">
