Commit message: Changed the reference location of meshes

File: rover/simulation/urdfs/rover.urdf (robot description, URDF)
Before this commit: robot rover, 12 links, 11 joints
Links:
- link chassis: geometry collision mesh filename=package://rover/rover/simulation/meshes/rover_meshes/chassi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; visual mesh filename=package://rover/rover/simulation/meshes/rover_meshes/chassi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
- link front_left_wheel: geometry collision mesh filename=package://rover/rover/simulation/meshes/rover_meshes/wheel_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; visual mesh filename=package://rover/rover/simulation/meshes/rover_meshes/wheel_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
- link front_right_wheel: geometry collision mesh filename=package://rover/rover/simulation/meshes/rover_meshes/wheel_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; visual mesh filename=package://rover/rover/simulation/meshes/rover_meshes/wheel_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
- link left_rocker: geometry collision mesh filename=package://rover/rover/simulation/meshes/rover_meshes/rocker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; visual mesh filename=package://rover/rover/simulation/meshes/rover_meshes/rocker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
- link lidar_link: geometry collision mesh filename=package://rover/rover/simulation/meshes/rover_meshes/os1_64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; visual mesh filename=package://rover/rover/simulation/meshes/rover_meshes/os1_64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
- link middle_left_wheel: geometry collision mesh filename=package://rover/rover/simulation/meshes/rover_meshes/wheel_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; visual mesh filename=package://rover/rover/simulation/meshes/rover_meshes/wheel_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
- link middle_right_wheel: geometry collision mesh filename=package://rover/rover/simulation/meshes/rover_meshes/wheel_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; visual mesh filename=package://rover/rover/simulation/meshes/rover_meshes/wheel_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
- link rear_left_wheel: geometry collision mesh filename=package://rover/rover/simulation/meshes/rover_meshes/wheel_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; visual mesh filename=package://rover/rover/simulation/meshes/rover_meshes/wheel_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
- link rear_right_wheel: geometry collision mesh filename=package://rover/rover/simulation/meshes/rover_meshes/wheel_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; visual mesh filename=package://rover/rover/simulation/meshes/rover_meshes/wheel_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
- link right_rocker: geometry collision mesh filename=package://rover/simulation/meshes/rover_meshes/rocker_1.STL; visual mesh filename=package://rover/rover/simulation/meshes/rover_meshes/rocker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

Commit message: move_base implemented on simulation.work needed

File: rover/simulation/urdfs/rover.urdf (robot description, URDF)
Before this commit: robot rover, 12 links, 11 joints
Links:
- link right_rocker: geometry collision mesh filename=package://rover/rover/simulation/meshes/rover_meshes/rocker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; visual mesh filename=package://rover/rover/simulation/meshes/rover_meshes/rocker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
