Commit message: Fixed chassis rotation error.

File: rover/simulation/urdf/Rover.urdf (robot description, URDF)
Before this commit: robot Rover, 9 links, 8 joints
Links:
- removed link rocker_1
- removed link rocker_2
- removed link wheel_1
- removed link wheel_2
- removed link wheel_3
- removed link wheel_4
- removed link wheel_5
- removed link wheel_6
- added link front_left_wheel, mass 3.71098880202612; collision mesh filename=package://rover/meshes/wheel_4.STL; visual mesh filename=package://rover/meshes/wheel_4.STL
- added link front_right_wheel, mass 3.71098878156725; collision mesh filename=package://rover/meshes/wheel_1.STL; visual mesh filename=package://rover/meshes/wheel_1.STL
- added link left_rocker, mass 0.702057959029149; collision mesh filename=package://rover/meshes/rocker_2.STL; visual mesh filename=package://rover/meshes/rocker_2.STL
- added link middle_left_wheel, mass 3.7109887931054; collision mesh filename=package://rover/meshes/wheel_5.STL; visual mesh filename=package://rover/meshes/wheel_5.STL
- added link middle_right_wheel, mass 3.71098876791251; collision mesh filename=package://rover/meshes/wheel_3.STL; visual mesh filename=package://rover/meshes/wheel_3.STL
- added link rear_left_wheel, mass 3.71098880708039; collision mesh filename=package://rover/meshes/wheel_6.STL; visual mesh filename=package://rover/meshes/wheel_6.STL
- added link rear_right_wheel, mass 3.71098882585926; collision mesh filename=package://rover/meshes/wheel_2.STL; visual mesh filename=package://rover/meshes/wheel_2.STL
- added link right_rocker, mass 0.702057959029176; collision mesh filename=package://rover/meshes/rocker_1.STL; visual mesh filename=package://rover/meshes/rocker_1.STL
- link chassis: geometry collision mesh filename=package://rover/meshes/chassis.STL; visual mesh filename=package://rover/meshes/chassis.STL
Joints:
- removed joint joint_1
- removed joint joint_2
- removed joint joint_3
- removed joint joint_4
- removed joint joint_5
- removed joint joint_6
- removed joint joint_7
- removed joint joint_8
- added joint chassis_left_rocker_joint: type fixed, parent chassis, child left_rocker, origin xyz=0.257280649253525 0.686809397997044 0.442407585082231 rpy=3.14159265358979 0 0, axis 0 1 0
- added joint chassis_right_rocker_joint: type fixed, parent chassis, child right_rocker, origin xyz=0.256227202845866 0.104049397997044 0.442431681089809 rpy=3.14159265358979 0 0, axis 0 1 0
- added joint front_left_wheel_joint: type continuous, parent left_rocker, child front_left_wheel, origin xyz=0.550522165589643 -0.128635200000009 0.363405762447953 rpy=0 0 0, axis 0 1 0
- added joint front_right_wheel_joint: type continuous, parent right_rocker, child front_right_wheel, origin xyz=0.566011190291999 0.1316352 0.343614113670245 rpy=0 0 0, axis 0 1 0
- added joint middle_left_wheel_joint: type continuous, parent left_rocker, child middle_left_wheel, origin xyz=-0.00926565490461811 -0.128635699999999 0.348270005795649 rpy=0 0 0, axis 0 1 0
- added joint middle_right_wheel_joint: type continuous, parent right_rocker, child middle_right_wheel, origin xyz=0.00389311933816788 0.135634699999995 0.348264389277544 rpy=0 0 0, axis 0 1 0
- added joint rear_left_wheel_joint: type continuous, parent left_rocker, child rear_left_wheel, origin xyz=-0.585325281230279 -0.124635699999999 0.308803919717537 rpy=0 0 0, axis 0 1 0
- added joint rear_right_wheel_joint: type continuous, parent right_rocker, child rear_right_wheel, origin xyz=-0.569418798760428 0.1316347 0.337858198560885 rpy=0 0 0, axis 0 1 0

Commit message: Fixed file paths in launch file.

File: rover/simulation/urdf/Rover.urdf (robot description, URDF)
Before this commit: robot rover, 9 links, 8 joints
Links:
- link chassis: geometry collision mesh filename=package://rover/rover/simulation/meshes/chassis.STL; visual mesh filename=package://rover/rover/simulation/meshes/chassis.STL
- link front_left_wheel: geometry collision mesh filename=package://rover/rover/simulation/meshes/wheel_4.STL; visual mesh filename=package://rover/rover/simulation/meshes/wheel_4.STL
- link front_right_wheel: geometry collision mesh filename=package://rover/rover/simulation/meshes/wheel_1.STL; visual mesh filename=package://rover/rover/simulation/meshes/wheel_1.STL
- link left_rocker: geometry collision mesh filename=package://rover/rover/simulation/meshes/rocker_2.STL; visual mesh filename=package://rover/rover/simulation/meshes/rocker_2.STL
- link middle_left_wheel: geometry collision mesh filename=package://rover/rover/simulation/meshes/wheel_5.STL; visual mesh filename=package://rover/rover/simulation/meshes/wheel_5.STL
- link middle_right_wheel: geometry collision mesh filename=package://rover/rover/simulation/meshes/wheel_3.STL; visual mesh filename=package://rover/rover/simulation/meshes/wheel_3.STL
- link rear_left_wheel: geometry collision mesh filename=package://rover/rover/simulation/meshes/wheel_6.STL; visual mesh filename=package://rover/rover/simulation/meshes/wheel_6.STL
- link rear_right_wheel: geometry collision mesh filename=package://rover/rover/simulation/meshes/wheel_2.STL; visual mesh filename=package://rover/rover/simulation/meshes/wheel_2.STL
- link right_rocker: geometry collision mesh filename=package://rover/simulation/meshes/rocker_1.STL; visual mesh filename=package://rover/rover/simulation/meshes/rocker_1.STL

Commit message: These files have IMU, GPS, Lidar and Odometry integrated on the real rover

File: rover/simulation/urdf/Rover.urdf (robot description, URDF)
Before this commit: robot rover, 9 links, 8 joints
Links:
- added link gps_link, mass 1e-5; collision box size=0.05 0.05 0.05; visual box size=0.05 0.05 0.05
- added link imu_link, mass 1e-5; collision box size=0.05 0.05 0.05; visual box size=0.05 0.05 0.05
- added link lidar_link, mass 0.425; collision mesh filename=package://rover/rover/simulation/meshes/os1_64.stl; visual mesh filename=package://rover/rover/simulation/meshes/os1_64.stl
Joints:
- added joint gps_joint: type fixed, parent chassis, child gps_link, origin xyz=0.0 0 0.278189004081027 rpy=0 0 0, axis 0 0 0
- added joint imu_joint: type fixed, parent chassis, child imu_link, origin xyz=0.0 0 0.0 rpy=1.5707963267949 0 0, axis 0 0 0
- added joint lidar_joint: type fixed, parent chassis, child lidar_link, origin xyz=0.0 0 0.278189004081027 rpy=0 0 0, axis 0 0 0
