Commit message: commiting eveyrthing so I can debug on laptop lol

File: rover/simulation/urdfs/Arm_2023/Arm_2023_gazebo.xacro (robot description, xacro)
@@ -1,5 +1,7 @@
 <?xml version="1.0" ?>
-<robot name="Arm_2023" xmlns:xacro="http://www.ros.org/wiki/xacro">
+<robot name="arm_2023" xmlns:xacro="http://www.ros.org/wiki/xacro">
 <xacro:include filename="$(find rover)/rover/simulation/urdfs/Arm_2023/materials.xacro" />
+<xacro:include filename="$(find rover)/rover/simulation/urdfs/Arm_2023/Arm_2023.trans" />
+<xacro:include filename="$(find rover)/rover/simulation/urdfs/Arm_2023/Arm_2023.gazebo" />
 <link name="base_link">
   <inertial>
@@ -22,5 +24,4 @@
   </collision>
 </link>
-<!-- Target Position Arm -->
 <link name="Link_2">
   <inertial>
@@ -236,5 +237,5 @@
 </joint>
 <joint name="Joint_3" type="continuous">
-  <origin xyz="0.0 0.0 0.365" rpy="-1.57 0 0"/>
+  <origin xyz="0.0 0.0 0.365" rpy="0 0 0"/>
   <parent link="Link_2"/>
   <child link="Link_3"/>
@@ -282,263 +283,9 @@
   <axis xyz="-1.0 0.0 0.0"/>
 </joint>
-<!-- Real Arm -->
-<link name="Real_Link_2">
-  <inertial>
-    <origin xyz="0.025 -3.469446951953614e-17 0.18250000000000027" rpy="0 0 0"/>
-    <mass value="1.86067089388539"/>
-    <inertia ixx="0.02649" iyy="0.026465" izz="0.001376" ixy="-0.0" iyz="0.0" ixz="-0.0"/>
-  </inertial>
-  <visual>
-    <origin xyz="-0.025 -0.043125 -0.1039" rpy="0 0 0"/>
-    <geometry>
-      <mesh filename="package://rover/rover/simulation/meshes/Arm_2023/Link_2_1.stl" scale="0.001 0.001 0.001"/>
-    </geometry>
-    <material name="sky-blue"/>
-  </visual>
-  <collision>
-    <origin xyz="-0.025 -0.043125 -0.1039" rpy="0 0 0"/>
-    <geometry>
-      <mesh filename="package://rover/rover/simulation/meshes/Arm_2023/Link_2_1.stl" scale="0.001 0.001 0.001"/>
-    </geometry>
-  </collision>
-</link>
-<link name="Real_Link_3">
-  <inertial>
-    <origin xyz="0.03437499999999986 -0.04852387230509649 0.01494234846228587" rpy="0 0 0"/>
-    <mass value="0.4930537063853911"/>
-    <inertia ixx="0.000808" iyy="0.000697" izz="0.001059" ixy="0.0" iyz="0.000147" ixz="0.0"/>
-  </inertial>
-  <visual>
-    <origin xyz="-0.025 -0.043125 -0.4689" rpy="0 0 0"/>
-    <geometry>
-      <mesh filename="package://rover/rover/simulation/meshes/Arm_2023/Link_3_1.stl" scale="0.001 0.001 0.001"/>
-    </geometry>
-    <material name="sky-blue"/>
-  </visual>
-  <collision>
-    <origin xyz="-0.025 -0.043125 -0.4689" rpy="0 0 0"/>
-    <geometry>
-      <mesh filename="package://rover/rover/simulation/meshes/Arm_2023/Link_3_1.stl" scale="0.001 0.001 0.001"/>
-    </geometry>
-  </collision>
-</link>
-<link name="Real_Link_4">
-  <inertial>
-    <origin xyz="-4.544770722816893e-05 5.898059818321144e-17 0.13249483155448072" rpy="0 0 0"/>
-    <mass value="1.3362092993202992"/>
-    <inertia ixx="0.010972" iyy="0.01038" izz="0.00176" ixy="0.0" iyz="0.0" ixz="-5e-06"/>
-  </inertial>
-  <visual>
-    <origin xyz="-0.059375 0.025375 -0.5139" rpy="0 0 0"/>
-    <geometry>
-      <mesh filename="package://rover/rover/simulation/meshes/Arm_2023/Link_4_1.stl" scale="0.001 0.001 0.001"/>
-    </geometry>
-    <material name="sky-blue"/>
-  </visual>
-  <collision>
-    <origin xyz="-0.059375 0.025375 -0.5139" rpy="0 0 0"/>
-    <geometry>
-      <mesh filename="package://rover/rover/simulation/meshes/Arm_2023/Link_4_1.stl" scale="0.001 0.001 0.001"/>
-    </geometry>
-  </collision>
-</link>
-<link name="Real_Link_5">
-  <inertial>
-    <origin xyz="-0.024457508265359702 0.028875000000000362 -0.00023164099942307725" rpy="0 0 0"/>
-    <mass value="1.03093485941646"/>
-    <inertia ixx="0.000373" iyy="0.001033" izz="0.001033" ixy="0.0" iyz="0.0" ixz="-8e-06"/>
-  </inertial>
-  <visual>
-    <origin xyz="-0.0667 0.05425 -0.790676" rpy="0 0 0"/>
-    <geometry>
-      <mesh filename="package://rover/rover/simulation/meshes/Arm_2023/Link_5_1.stl" scale="0.001 0.001 0.001"/>
-    </geometry>
-    <material name="sky-blue"/>
-  </visual>
-  <collision>
-    <origin xyz="-0.0667 0.05425 -0.790676" rpy="0 0 0"/>
-    <geometry>
-      <mesh filename="package://rover/rover/simulation/meshes/Arm_2023/Link_5_1.stl" scale="0.001 0.001 0.001"/>
-    </geometry>
-  </collision>
-</link>
-<link name="Real_Link_1">
-  <inertial>
-    <origin xyz="-7.179673522372809e-14 -0.00017173384764001404 0.045632894964534494" rpy="0 0 0"/>
-    <mass value="0.4382416946666404"/>
-    <inertia ixx="0.000836" iyy="0.000966" izz="0.000383" ixy="0.0" iyz="4e-06" ixz="-0.0"/>
-  </inertial>
-  <visual>
-    <origin xyz="-0.05 -0.04 -0.00625" rpy="0 0 0"/>
-    <geometry>
-      <mesh filename="package://rover/rover/simulation/meshes/Arm_2023/Link_1_1.stl" scale="0.001 0.001 0.001"/>
-    </geometry>
-    <material name="sky-blue"/>
-  </visual>
-  <collision>
-    <origin xyz="-0.05 -0.04 -0.00625" rpy="0 0 0"/>
-    <geometry>
-      <mesh filename="package://rover/rover/simulation/meshes/Arm_2023/Link_1_1.stl" scale="0.001 0.001 0.001"/>
-    </geometry>
-  </collision>
-</link>
-<link name="Real_Link_6">
-  <inertial>
-    <origin xyz="0.0007934173167834443 -0.0006657561778822887 0.04453519096184422" rpy="0 0 0"/>
-    <mass value="3.060647277391577"/>
-    <inertia ixx="0.003765" iyy="0.003842" izz="0.003929" ixy="0.000217" iyz="7.2e-05" ixz="-8.6e-05"/>
-  </inertial>
-  <visual>
-    <origin xyz="-0.059375 0.025375 -0.815676" rpy="0 0 0"/>
-    <geometry>
-      <mesh filename="package://rover/rover/simulation/meshes/Arm_2023/Link_6_1.stl" scale="0.001 0.001 0.001"/>
-    </geometry>
-    <material name="sky-blue"/>
-  </visual>
-  <collision>
-    <origin xyz="-0.059375 0.025375 -0.815676" rpy="0 0 0"/>
-    <geometry>
-      <mesh filename="package://rover/rover/simulation/meshes/Arm_2023/Link_6_1.stl" scale="0.001 0.001 0.001"/>
-    </geometry>
-  </collision>
-</link>
-<link name="Real_Link_7">
-  <inertial>
-    <origin xyz="-0.0017868967775850602 -0.005028096180721024 0.04636811966902066" rpy="0 0 0"/>
-    <mass value="0.07042769953386388"/>
-    <inertia ixx="9.8e-05" iyy="9.8e-05" izz="1e-06" ixy="0.0" iyz="3e-06" ixz="-4e-06"/>
-  </inertial>
-  <visual>
-    <origin xyz="0.007887 -0.037592 -0.899176" rpy="0 0 0"/>
-    <geometry>
-      <mesh filename="package://rover/rover/simulation/meshes/Arm_2023/Link_7_1.stl" scale="0.001 0.001 0.001"/>
-    </geometry>
-    <material name="sky-blue"/>
-  </visual>
-  <collision>
-    <origin xyz="0.007887 -0.037592 -0.899176" rpy="0 0 0"/>
-    <geometry>
-      <mesh filename="package://rover/rover/simulation/meshes/Arm_2023/Link_7_1.stl" scale="0.001 0.001 0.001"/>
-    </geometry>
-  </collision>
-</link>
-<link name="Real_Camera_link">
-  <inertial>
-    <origin xyz="-0.01999999999995162 3.608224830031759e-16 0.0008309682104639116" rpy="0 0 0"/>
-    <mass value="0.5216667986958432"/>
-    <inertia ixx="0.000144" iyy="0.000144" izz="0.000135" ixy="0.0" iyz="0.0" ixz="-0.0"/>
-  </inertial>
-  <visual>
-    <origin xyz="0.015625 0.025375 -0.79" rpy="0 0 0"/>
-    <geometry>
-      <mesh filename="package://rover/rover/simulation/meshes/Arm_2023/Camera_link_1.stl" scale="0.001 0.001 0.001"/>
-    </geometry>
-    <material name="sky-blue"/>
-  </visual>
-  <collision>
-    <origin xyz="0.015625 0.025375 -0.79" rpy="0 0 0"/>
-    <geometry>
-      <mesh filename="package://rover/rover/simulation/meshes/Arm_2023/Camera_link_1.stl" scale="0.001 0.001 0.001"/>
-    </geometry>
-  </collision>
-</link>
-<link name="Real_Link_8">
-  <inertial>
-    <origin xyz="-0.002703449377635364 0.004600114186135835 0.04636811966902088" rpy="0 0 0"/>
-    <mass value="0.07042769953386384"/>
-    <inertia ixx="9.8e-05" iyy="9.8e-05" izz="1e-06" ixy="-0.0" iyz="1e-06" ixz="5e-06"/>
-  </inertial>
-  <visual>
-    <origin xyz="-0.150846 0.014323 -0.899176" rpy="0 0 0"/>
-    <geometry>
-      <mesh filename="package://rover/rover/simulation/meshes/Arm_2023/Link_8_1.stl" scale="0.001 0.001 0.001"/>
-    </geometry>
-    <material name="sky-blue"/>
-  </visual>
-  <collision>
-    <origin xyz="-0.150846 0.014323 -0.899176" rpy="0 0 0"/>
-    <geometry>
-      <mesh filename="package://rover/rover/simulation/meshes/Arm_2023/Link_8_1.stl" scale="0.001 0.001 0.001"/>
-    </geometry>
-  </collision>
-</link>
-<link name="Real_Link_9">
-  <inertial>
-    <origin xyz="0.005000000000008033 0.001863066826134921 0.04636811966902088" rpy="0 0 0"/>
-    <mass value="0.07042769953386384"/>
-    <inertia ixx="9.8e-05" iyy="9.8e-05" izz="1e-06" ixy="-0.0" iyz="-5e-06" ixz="0.0"/>
-  </inertial>
-  <visual>
-    <origin xyz="-0.054375 0.117375 -0.899176" rpy="0 0 0"/>
-    <geometry>
-      <mesh filename="package://rover/rover/simulation/meshes/Arm_2023/Link_9_1.stl" scale="0.001 0.001 0.001"/>
-    </geometry>
-    <material name="sky-blue"/>
-  </visual>
-  <collision>
-    <origin xyz="-0.054375 0.117375 -0.899176" rpy="0 0 0"/>
-    <geometry>
-      <mesh filename="package://rover/rover/simulation/meshes/Arm_2023/Link_9_1.stl" scale="0.001 0.001 0.001"/>
-    </geometry>
-  </collision>
-</link>
-<joint name="Real_Joint_1" type="continuous">
-  <origin xyz="0.05 0.04 0.00625" rpy="0 0 0"/>
-  <parent link="base_link"/>
-  <child link="Real_Link_1"/>
-  <axis xyz="0.0 0.0 1.0"/>
-</joint>
-<joint name="Real_Joint_2" type="continuous">
-  <origin xyz="-0.025 0.003125 0.09765" rpy="-1.57 0 0"/>
-  <parent link="Real_Link_1"/>
-  <child link="Real_Link_2"/>
-  <axis xyz="1.0 0.0 -0.0"/>
-</joint>
-<joint name="Real_Joint_3" type="continuous">
-  <origin xyz="0.0 0.0 0.365" rpy="-1.57 0 0"/>
-  <parent link="Real_Link_2"/>
-  <child link="Real_Link_3"/>
-  <axis xyz="1.0 -0.0 0.0"/>
-</joint>
-<joint name="Real_Joint_4" type="continuous">
-  <origin xyz="0.034375 -0.0685 0.045" rpy="0 0 -1.57"/>
-  <parent link="Real_Link_3"/>
-  <child link="Real_Link_4"/>
-  <axis xyz="0.0 0.0 1.0"/>
-</joint>
-<joint name="Real_Joint_5" type="continuous">
-  <origin xyz="0.007325 -0.028875 0.276776" rpy="0 0 0"/>
-  <parent link="Real_Link_4"/>
-  <child link="Real_Link_5"/>
-  <axis xyz="-0.0 1.0 -0.0"/>
-</joint>
-<joint name="Real_Joint_6" type="continuous">
-  <origin xyz="-0.007325 0.028875 0.025" rpy="0 0 0"/>
-  <parent link="Real_Link_5"/>
-  <child link="Real_Link_6"/>
-  <axis xyz="-0.0 0.0 -1.0"/>
-</joint>
-<joint name="Real_Joint_7" type="continuous">
-  <origin xyz="-0.067262 0.062967 0.0835" rpy="0 0 0"/>
-  <parent link="Real_Link_6"/>
-  <child link="Real_Link_7"/>
-  <axis xyz="0.642788 0.766044 0.0"/>
-</joint>
-<joint name="Real_Camera_Joint" type="fixed">
-  <origin xyz="-0.082325 0.028875 -0.000676" rpy="0 0 0"/>
-  <parent link="Real_Link_5"/>
-  <child link="Real_Camera_link"/>
-</joint>
-<joint name="Real_Joint_8" type="continuous">
-  <origin xyz="0.091471 0.011052 0.0835" rpy="0 0 0"/>
-  <parent link="Real_Link_6"/>
-  <child link="Real_Link_8"/>
-  <axis xyz="0.173648 -0.984808 -0.0"/>
-</joint>
-<joint name="Real_Joint_9" type="continuous">
-  <origin xyz="-0.005 -0.092 0.0835" rpy="0 0 0"/>
-  <parent link="Real_Link_6"/>
-  <child link="Real_Link_9"/>
-  <axis xyz="-1.0 0.0 0.0"/>
+<!-- Fix arm in place -->
+<link name="world"/>
+<joint name="fixed" type="fixed">
+  <parent link="world"/>
+  <child link="base_link"/>
 </joint>
 </robot>

Commit message: ik should be ready for gazebo, bug switching b/w manual and ik

File: rover/simulation/urdfs/Arm_2023/Arm_2023_gazebo.xacro (robot description, xacro)
@@ -231,5 +231,5 @@
 </joint>
 <joint name="Joint_2" type="continuous">
-  <origin xyz="-0.025 0.003125 0.09765" rpy="-1.57 0 0"/>
+  <origin xyz="-0.025 0.003125 0.09765" rpy="0 0 0"/>
   <parent link="Link_1"/>
   <child link="Link_2"/>
@@ -237,5 +237,5 @@
 </joint>
 <joint name="Joint_3" type="continuous">
-  <origin xyz="0.0 0.0 0.365" rpy="0 0 0"/>
+  <origin xyz="0.0 0.0 0.365" rpy="-1.57 0 0"/>
   <parent link="Link_2"/>
   <child link="Link_3"/>
@@ -252,5 +252,5 @@
   <parent link="Link_4"/>
   <child link="Link_5"/>
-  <axis xyz="-0.0 1.0 -0.0"/>
+  <axis xyz="-0.0 -1.0 -0.0"/>
 </joint>
 <joint name="Joint_6" type="continuous">

Commit message: Fixed Gazebo Funkyness
- gazebo does not like it when the angles are coming in too fast
- gazebo does not like it when ik and arm_controller are running at diff speeds
- just run both at 100Hz to be safe

File: rover/simulation/urdfs/Arm_2023/Arm_2023_gazebo.xacro (robot description, xacro)
@@ -252,5 +252,5 @@
   <parent link="Link_4"/>
   <child link="Link_5"/>
-  <axis xyz="-0.0 -1.0 -0.0"/>
+  <axis xyz="-0.0 1.0 -0.0"/>
 </joint>
 <joint name="Joint_6" type="continuous">

Commit message: arm visualization node now does all work to visualize in gazebo

File: rover/simulation/urdfs/Arm_2023/Arm_2023_gazebo.xacro (robot description, xacro)
@@ -252,5 +252,5 @@
   <parent link="Link_4"/>
   <child link="Link_5"/>
-  <axis xyz="-0.0 1.0 -0.0"/>
+  <axis xyz="-0.0 -1.0 -0.0"/>
 </joint>
 <joint name="Joint_6" type="continuous">

Commit message: added required plugins in to gazebo urdf

File: rover/simulation/urdfs/Arm_2023/Arm_2023_gazebo.xacro (robot description, xacro)
@@ -289,4 +289,52 @@
   <child link="base_link"/>
 </joint>
+<!-- Camera Stuff -->
+<link name="camera_optical"/>
+<joint name="optical_joint" type="fixed">
+  <parent link="Camera_link"/>
+  <child link="camera_optical"/>
+  <origin xyz="0 0 0" rpy="-1.571 0 -1.571"/>
+</joint>
+<gazebo reference="Camera_link">
+  <sensor name="camera" type="depth">
+    <update_rate>20</update_rate>
+    <camera>
+      <horizontal_fov>1.5</horizontal_fov>
+      <image>
+        <width>640</width>
+        <height>480</height>
+        <format>R8G8B8</format>
+      </image>
+      <clip>
+        <near>0.05</near>
+        <far>3</far>
+      </clip>
+    </camera>
+    <plugin name="camera_plugin" filename="libgazebo_ros_openni_kinect.so">
+      <baseline>0.2</baseline>
+      <alwaysOn>true</alwaysOn>
+      <updateRate>1.0</updateRate>
+      <cameraName>camera_ir</cameraName>
+      <imageTopicName>/camera/color/image_raw</imageTopicName>
+      <cameraInfoTopicName>/camera/color/camera_info</cameraInfoTopicName>
+      <depthImageTopicName>/camera/depth/image_raw</depthImageTopicName>
+      <depthImageInfoTopicName>/camera/depth/camera_info</depthImageInfoTopicName>
+      <pointCloudTopicName>/camera/depth/points</pointCloudTopicName>
+      <frameName>camera_optical</frameName> <!-- name of link -->
+      <pointCloudCutoff>0</pointCloudCutoff>
+      <pointCloudCutoffMax>3.5</pointCloudCutoffMax>
+      <distortionK1>0</distortionK1>
+      <distortionK2>0</distortionK2>
+      <distortionK3>0</distortionK3>
+      <distortionT1>0</distortionT1>
+      <distortionT2>0</distortionT2>
+      <CxPrime>0</CxPrime>
+      <Cx>0</Cx>
+      <Cy>0</Cy>
+      <focalLength>0</focalLength>
+      <hackBaseline>0</hackBaseline>
+    </plugin>
+  </sensor>
+</gazebo>
 <!-- Gazebo Plugins-->
 <gazebo>
@@ -294,4 +342,20 @@
     <robotNamespace>/arm</robotNamespace>
   </plugin>
+  <plugin name="gazebo_grasp_fix" filename="libgazebo_grasp_fix.so">
+        <arm>
+           <arm_name>arm</arm_name>
+           <palm_link>Link_6</palm_link>
+           <gripper_link>Link_7</gripper_link>
+           <gripper_link>Link_8</gripper_link>
+           <gripper_link>Link_9</gripper_link>
+        </arm>
+       <forces_angle_tolerance>100</forces_angle_tolerance>
+       <update_rate>4</update_rate>
+       <grip_count_threshold>4</grip_count_threshold>
+       <max_grip_count>8</max_grip_count>
+       <release_tolerance>0.005</release_tolerance>
+       <disable_collisions_on_attach>false</disable_collisions_on_attach>
+       <contact_topic>__default_topic__</contact_topic>
+    </plugin>
 </gazebo>
 </robot>

Commit message: got gazebo 3D camera working with new urdf

File: rover/simulation/urdfs/Arm_2023/Arm_2023_gazebo.xacro (robot description, xacro)
@@ -267,5 +267,5 @@
 </joint>
 <joint name="Camera_Joint" type="fixed">
-  <origin xyz="-0.082325 0.028875 -0.000676" rpy="0 0 0"/>
+  <origin xyz="-0.082325 0.028875 -0.000676" rpy="3.14 -1.571 -1.571"/>
   <parent link="Link_5"/>
   <child link="Camera_link"/>
