Commit message: CHanges to make shit work

File: rover/simulation/urdfs/Arm_CIRC_2024/URDF.xacro (robot description, xacro)
@@ -261,5 +261,5 @@
   <axis xyz="-0.0 0.0 1.0"/>
 </joint>
-<joint name="Joint_7" type="continuous">
+<joint name="Joint_7" type="fixed">
   <origin xyz="-0.067262 0.062967 0.064" rpy="0 0 0"/>
   <parent link="link_6"/>
@@ -272,5 +272,5 @@
   <child link="link_8"/>
 </joint>
-<joint name="Joint_8" type="continuous">
+<joint name="Joint_8" type="fixed">
   <origin xyz="0.091471 0.011052 0.064" rpy="0 0 0"/>
   <parent link="link_6"/>
@@ -278,5 +278,5 @@
   <axis xyz="0.173648 -0.984808 -0.0"/>
 </joint>
-<joint name="Joint_9" type="continuous">
+<joint name="Joint_9" type="fixed">
   <origin xyz="-0.005 -0.092 0.064" rpy="0 0 0"/>
   <parent link="link_6"/>
@@ -521,5 +521,5 @@
   <axis xyz="-0.0 0.0 1.0"/>
 </joint>
-<joint name="Real_Joint_7" type="continuous">
+<joint name="Real_Joint_7" type="fixed">
   <origin xyz="-0.067262 0.062967 0.064" rpy="0 0 0"/>
   <parent link="real_link_6"/>
@@ -532,5 +532,5 @@
   <child link="real_link_8"/>
 </joint>
-<joint name="Real_Joint_8" type="continuous">
+<joint name="Real_Joint_8" type="fixed">
   <origin xyz="0.091471 0.011052 0.064" rpy="0 0 0"/>
   <parent link="real_link_6"/>
@@ -538,5 +538,5 @@
   <axis xyz="0.173648 -0.984808 -0.0"/>
 </joint>
-<joint name="Real_Joint_9" type="continuous">
+<joint name="Real_Joint_9" type="fixed">
   <origin xyz="-0.005 -0.092 0.064" rpy="0 0 0"/>
   <parent link="real_link_6"/>

Commit message: fixed some viz stuff

File: rover/simulation/urdfs/Arm_CIRC_2024/URDF.xacro (robot description, xacro)
@@ -244,5 +244,5 @@
 </joint>
 <joint name="Joint_4" type="continuous">
-  <origin xyz="0.034375 -0.1 0.045" rpy="0 0 -1.57"/>
+  <origin xyz="0.034375 -0.1 0.045" rpy="0 0 1.57"/>
   <parent link="link_3"/>
   <child link="link_4"/>
@@ -253,5 +253,5 @@
   <parent link="link_4"/>
   <child link="link_5"/>
-  <axis xyz="-0.0 1.0 -0.0"/>
+  <axis xyz="-0.0 -1.0 -0.0"/>
 </joint>
 <joint name="Joint_6" type="continuous">
@@ -259,5 +259,5 @@
   <parent link="link_5"/>
   <child link="link_6"/>
-  <axis xyz="-0.0 0.0 1.0"/>
+  <axis xyz="-0.0 0.0 -1.0"/>
 </joint>
 <joint name="Joint_7" type="fixed">
